File: Ad_Fontes/Ad_Fontes.kicad_sch (KiCad schematic)
At the start: 14 parts, among them J1 AVR-ISP-6, SW1 SW_SPST, SW2 SW_SPDT, U1 ATTINY1616-MFR

Commit message: Cleaning up and adding documention
Other:
- note added: "Power Switch"
- note added: "Press Button"
- note removed: "Button"
- company: Aerospace Village -> Ad Fontes
- title: Moonlighter -> Ad Fontes STEM Event
- moved on the sheet: BT1, D1, D2, D3, D4, J1, R1, R2, R3, R4, SW2
